File: hardware/neopico-hd/neopico-hd.kicad_sch (KiCad schematic)
At the start: 12 parts, among them J1 HDMI_A, U1 SN74LVC2G14DBV, U2 SN74LVC2G14DBV, U3 SN74LVC245APW, U4 SN74LVC245APW, U5 SN74LVC245APW

Commit message: Update schematics
Parts:
- added C6: C_Polarized, Capacitor_THT:CP_Radial_D5.0mm_P2.00mm, symbol Device:C_Polarized
- added C7: 0.1u, custom_components:SM0603_Capa_libcms, symbol Device:C
- added D1: SS14, Diode_SMD:D_SMA, symbol Diode:SS14
- added F1: Polyfuse, symbol Device:Polyfuse
- added FB1: FerriteBead, symbol Device:FerriteBead
- added U6, U7: ESD224DQA, Package_DFN_QFN:Diodes_UDFN-10_1.0x2.5mm_P0.5mm, symbol Power_Protection:ESD224DQA
- J1: footprint (none) -> Connector_Video:HDMI_A_Molex_208658-1001_Horizontal
Connections:
- net VCC is gone; now on net +3V3: C1.1, C2.1, C3.1, C4.1, C5.1, U1.5 (V_{CC}), U2.5 (V_{CC}), U3.20 (VCC), U4.20 (VCC), U5.20 (VCC)
- net +3V3: now also A1.55 (3V3)
- net +5V: now also C7.1; no longer A1.1 (VBUS)
- net BCK: now also A1.8 (GPIO2)
- net DAT: now also A1.6 (GPIO0)
- net GND: now also C6.2, C7.2
- net WS: now also A1.7 (GPIO1)
- net +5V FILTERED: now reaches A1.2 (VSYS)
- net +5V FILTERED: now also C6.1, F1.2
- net HDMI_CLK_N renamed D2+
- net D2+: now also U6.1; no longer J1.12 (CK-)
- net HDMI_CLK_P renamed D2-
- net D2-: now also U6.2; no longer J1.10 (CK+)
- net HTMI_D0_N renamed D1+
- net D1+: now also U6.4; no longer J1.9 (D0-)
- net HTMI_D0_P renamed D1-
- net D1-: now also U6.5; no longer J1.7 (D0+)
- net HTMI_D1_N renamed D0+
- net D0+: now also U7.1; no longer J1.6 (D1-)
- net HTMI_D1_P renamed D0-
- net D0-: now also U7.2; no longer J1.4 (D1+)
- net HTMI_D2_N renamed CLK+
- net CLK+: now also U7.4; no longer J1.3 (D2-)
- net HTMI_D2_P renamed CLK-
- net CLK-: now also U7.5; no longer J1.1 (D2+)
- new net: U6.3 (VSS), U6.8 (VSS)
- new net: F1.1, FB1.2
- new net: D1.1 (K), FB1.1
- new net: U7.3 (VSS), U7.8 (VSS)
- new net +5V MVS: D1.2 (A)
- new net HDMI_CLK+: J1.10 (CK+), U7.7
- new net HDMI_CLK-: J1.12 (CK-), U7.6
- new net HDMI_D0+: J1.7 (D0+), U7.10
- new net HDMI_D0-: J1.9 (D0-), U7.9
- new net HDMI_D1+: J1.4 (D1+), U6.7
- new net HDMI_D1-: J1.6 (D1-), U6.6
- new net HDMI_D2+: J1.1 (D2+), U6.10
- new net HDMI_D2-: J1.3 (D2-), U6.9
- no-connect marks 24 -> 31
Other:
- note added: "Power"
- moved on the sheet: A1, J1
