File: hardware/neopico-hd/neopico-hd.kicad_sch (KiCad schematic)
At the start: 22 parts, among them J1 HDMI_A, J2 Conn_02x05_Top_Bottom, J3 Audio, J4 Audio, J5 AUX, J6 Conn_01x02_Pin, U1 A_BUFF, U2 V_BUFF, U3 RG_LVS, U4 GB_LVS, U5 AV_LVS

Commit message: V1 PCB
Parts:
- removed J3: Audio, Connector_JST:JST_XA_B03B-XASK-1_1x03_P2.50mm_Vertical, symbol Connector_Generic:Conn_01x03
- added R1: 27K, Resistor_SMD:R_0805_2012Metric, symbol Device:R
- added SW1: MENU, Connector_Samtec_HPM_THT:Samtec_HPM-02-01-x-S_Straight_1x02_Pitch5.08mm, symbol Switch:SW_DIP_x01
- added SW2: BACK, Connector_Samtec_HPM_THT:Samtec_HPM-02-01-x-S_Straight_1x02_Pitch5.08mm, symbol Switch:SW_DIP_x01
- J5: footprint Connector_JST:JST_XA_B08B-XASK-1_1x08_P2.50mm_Vertical -> Connector_PinHeader_2.54mm:PinHeader_2x04_P2.54mm_Vertical
Connections:
- net +3V3: now also U3.1 (DIR), U4.1 (DIR), U5.1 (DIR), R1.1; no longer U3.19 (~{OE}), U4.19 (~{OE}), U5.19 (~{OE})
- net GND: now also A1.58 (GND), J1.2 (D2S), J1.5 (D1S), J1.8 (D0S), J1.SH, U3.19 (~{OE}), U4.19 (~{OE}), U5.19 (~{OE}), SW1.2, SW2.2; no longer A1.57 (AGND), U3.1 (DIR), U4.1 (DIR), U5.1 (DIR)
- net MVS_SHD: now also U4.9 (A8); no longer U5.8 (A7)
- net SHD: now also U4.11 (B8); no longer U5.12 (B7)
- net at A1.6 (GPIO0): now also J5.1 (Pin_1)
- net at A1.7 (GPIO1): now also J5.2 (Pin_2)
- net at A1.8 (GPIO2): now also J5.3 (Pin_3)
- net at A1.10 (GPIO4): now also J5.5 (Pin_5); no longer J5.2 (Pin_2)
- net at A1.11 (GPIO5): now also J5.6 (Pin_6); no longer J5.3 (Pin_3)
- net at A1.12 (GPIO6): now also J5.7 (Pin_7); no longer J5.4 (Pin_4)
- net at A1.13 (GPIO7): now also J5.8 (Pin_8); no longer J5.5 (Pin_5)
- net CEC_PICO: now reaches A1.14 (GPIO8)
- net CEC_PICO: now also J1.13 (CEC), R1.2; no longer J5.6 (Pin_6)
- net at A1.15 (GPIO9): no longer J5.7 (Pin_7)
- net at A1.16 (GPIO10): no longer J5.8 (Pin_8)
- net SW_MENU: now reaches A1.31 (GPIO25)
- net SW_MENU: now also SW1.1
- net SW_BACK: now reaches A1.32 (GPIO26)
- net SW_BACK: now also SW2.1
- net at A1.9 (GPIO3): now also J5.4 (Pin_4); no longer J5.1 (Pin_1)
- net DARK: no longer names the net of A1.51 (GPIO45)
- net DARK: no longer U5.11 (B8)
- net MVS_DARK: no longer names the net of J2.17 (Pin_17)
- net MVS_DARK: no longer U5.9 (A8)
- no-connect marks 24 -> 33
Other:
- moved on the sheet: J5

Commit message: Update hardware
Parts:
- added R2: 10K, Resistor_SMD:R_0805_2012Metric_Pad1.20x1.40mm_HandSolder, symbol Device:R
- C6: value C_Polarized -> 47u
Connections:
- net +5V: now also R2.1
- net GND: now also J1.11 (CKS)
- net at J1.19 (HPD): now also R2.2
- no-connect marks 33 -> 31
Other:
- moved on the sheet: R1
Changed lines of the file:
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@@
 	)
 	(no_connect
-		(at 254 87.63)
-	)
-	(no_connect
-		(at 266.7 97.79)
-	)
-	(no_connect
 		(at 228.6 43.18)
 	)
@@
 	(wire
 		(pts
-			(xy 246.38 72.39) (xy 241.3 72.39)
+			(xy 73.66 182.88) (xy 73.66 185.42)
 		)
 		(stroke
@@
 	(wire
 		(pts
-			(xy 73.66 182.88) (xy 73.66 185.42)
+			(xy 43.18 88.9) (xy 43.18 91.44)
 		)
 		(stroke
@@
 	(wire
 		(pts
-			(xy 43.18 88.9) (xy 43.18 91.44)
+			(xy 96.52 96.52) (xy 92.71 96.52)
 		)
 		(stroke
@@
 	(wire
 		(pts
-			(xy 96.52 96.52) (xy 92.71 96.52)
+			(xy 40.64 170.18) (xy 45.72 170.18)
 		)
 		(stroke
@@
 	(wire
 		(pts
-			(xy 40.64 170.18) (xy 45.72 170.18)
+			(xy 58.42 91.44) (xy 55.88 91.44)
 		)
 		(stroke
@@
 	(wire
 		(pts
-			(xy 58.42 91.44) (xy 55.88 91.44)
+			(xy 247.65 72.39) (xy 254 72.39)
 		)
 		(stroke
@@
 	(global_label "CEC_PICO"
 		(shape bidirectional)
-		(at 254 72.39 270)
+		(at 250.19 72.39 270)
 		(fields_autoplaced yes)
 		(effects
@@
 		)
 		(property "Intersheetrefs" "${INTERSHEET_REFS}"
-			(at 254 85.6184 90)
+			(at 250.19 85.6184 90)
 			(effects
 				(font
@@
 			)
 		)
-		(property "Value" "C_Polarized"
+		(property "Value" "47u"
 			(at 77.47 179.4509 0)
 			(effects
@@
 	(symbol
 		(lib_id "power:+3V3")
-		(at 241.3 72.39 180)
+		(at 240.03 72.39 0)
 		(unit 1)
 		(exclude_from_sim no)
@@
 		(dnp no)
 		(property "Reference" "#PWR035"
-			(at 241.3 68.58 0)
+			(at 240.03 76.2 0)
 			(effects
 				(font
@@
 		)
 		(property "Value" "+3V3"
-			(at 241.2999 76.2 90)
+			(at 240.0301 68.58 90)
 			(effects
 				(font
@@
 		)
 		(property "Footprint" ""
-			(at 241.3 72.39 0)
+			(at 240.03 72.39 0)
 			(effects
 				(font
@@
 		)
 		(property "Datasheet" ""
-			(at 241.3 72.39 0)
+			(at 240.03 72.39 0)
 			(effects
 				(font
@@
 		)
 		(property "Description" "Power symbol creates a global label with name \"+3V3\""
-			(at 241.3 72.39 0)
+			(at 240.03 72.39 0)
 			(effects
 				(font
@@
 	)
 	(symbol
+		(lib_id "power:+5V")
+		(at 246.38 87.63 90)
+		(unit 1)
+		(exclude_from_sim no)
+		(in_bom yes)
+		(on_board yes)
+		(dnp no)
+		(fields_autoplaced yes)
+		(property "Reference" "#PWR036"
+			(at 250.19 87.63 0)
+			(effects
+				(font
+					(size 1.27 1.27)
+				)
+				(hide yes)
+			)
+		)
+		(property "Value" "+5V"
+			(at 242.57 87.6299 90)
+			(effects
+				(font
+					(size 1.27 1.27)
+				)
+				(justify left)
+			)
+		)
+		(property "Footprint" ""
+			(at 246.38 87.63 0)
+			(effects
+				(font
+					(size 1.27 1.27)
+				)
+				(hide yes)
+			)
+		)
+		(property "Datasheet" ""
+			(at 246.38 87.63 0)
+			(effects
+				(font
+					(size 1.27 1.27)
+				)
+				(hide yes)
+			)
+		)
+		(property "Description" "Power symbol creates a global label with name \"+5V\""
+			(at 246.38 87.63 0)
+			(effects
+				(font
+					(size 1.27 1.27)
+				)
+				(hide yes)
+			)
+		)
+		(pin "1"
+		)
+		(instances
+			(project ""
+				(path "/e43af130-6d9a-4b98-bcf6-f3f51cb37ae8"
+					(reference "#PWR036")
+					(unit 1)
+				)
+			)
+		)
+	)
+	(symbol
 		(lib_id "Device:C")
 		(at 100.33 96.52 90)
@@
 	(symbol
 		(lib_id "Device:R")
-		(at 250.19 72.39 90)
+		(at 243.84 72.39 90)
 		(unit 1)
 		(exclude_from_sim no)
@@
 		(dnp no)
 		(property "Reference" "R1"
-			(at 250.698 75.184 90)
+			(at 244.348 75.184 90)
 			(effects
 				(font
@@
 		)
 		(property "Value" "27K"
-			(at 250.698 77.724 90)
+			(at 244.348 77.724 90)
 			(effects
 				(font
@@
 		)
 		(property "Footprint" "Resistor_SMD:R_0805_2012Metric"
-			(at 250.19 74.168 90)
+			(at 243.84 74.168 90)
 			(effects
 				(font
@@
 		)
 		(property "Datasheet" "~"
-			(at 250.19 72.39 0)
+			(at 243.84 72.39 0)
 			(effects
 				(font
@@
 		)
 		(property "Description" "Resistor"
-			(at 250.19 72.39 0)
+			(at 243.84 72.39 0)
 			(effects
 				(font
@@
 		(on_board yes)
 		(dnp no)
-		(fields_autoplaced yes)
 		(property "Reference" "#PWR032"
 			(at 259.08 104.14 0)
@@
 		)
 		(property "Value" "GND"
-			(at 259.08 102.87 0)
+			(at 266.7 102.87 90)
 			(effects
 				(font
@@
 	(symbol
 		(lib_id "power:GND")
+		(at 266.7 97.79 0)
+		(unit 1)
+		(exclude_from_sim no)
+		(in_bom yes)
+		(on_board yes)
+		(dnp no)
+		(property "Reference" "#PWR040"
+			(at 266.7 104.14 0)
+			(effects
+				(font
+					(size 1.27 1.27)
+				)
+				(hide yes)
+			)
+		)
+		(property "Value" "GND"
+			(at 259.08 102.87 90)
+			(effects
+				(font
+					(size 1.27 1.27)
+				)
+			)
+		)
+		(property "Footprint" ""
+			(at 266.7 97.79 0)
+			(effects
+				(font
+					(size 1.27 1.27)
+				)
+				(hide yes)
+			)
+		)
+		(property "Datasheet" ""
+			(at 266.7 97.79 0)
+			(effects
+				(font
+					(size 1.27 1.27)
+				)
+				(hide yes)
+			)
+		)
+		(property "Description" "Power symbol creates a global label with name \"GND\" , ground"
+			(at 266.7 97.79 0)
+			(effects
+				(font
+					(size 1.27 1.27)
+				)
+				(hide yes)
+			)
+		)
+		(pin "1"
+		)
+		(instances
+			(project "neopico-hd"
+				(path "/e43af130-6d9a-4b98-bcf6-f3f51cb37ae8"
+					(reference "#PWR040")
+					(unit 1)
+				)
+			)
+		)
+	)
+	(symbol
+		(lib_id "power:GND")
 		(at 182.88 33.02 270)
 		(unit 1)
@@
 	)
 	(symbol
+		(lib_id "Device:R")
+		(at 250.19 87.63 90)
+		(unit 1)
+		(exclude_from_sim no)
+		(in_bom yes)
+		(on_board yes)
+		(dnp no)
+		(property "Reference" "R2"
+			(at 250.444 90.424 90)
+			(effects
+				(font
+					(size 1.27 1.27)
+				)
+			)
+		)
+		(property "Value" "10K"
+			(at 250.698 92.964 90)
+			(effects
+				(font
+					(size 1.27 1.27)
+				)
+				(hide yes)
+			)
+		)
+		(property "Footprint" "Resistor_SMD:R_0805_2012Metric_Pad1.20x1.40mm_HandSolder"
+			(at 250.19 89.408 90)
+			(effects
+				(font
+					(size 1.27 1.27)
+				)
+				(hide yes)
+			)
+		)
+		(property "Datasheet" "~"
+			(at 250.19 87.63 0)
+			(effects
+				(font
+					(size 1.27 1.27)
+				)
+				(hide yes)
+			)
+		)
+		(property "Description" "Resistor"
+			(at 250.19 87.63 0)
+			(effects
+				(font
+					(size 1.27 1.27)
+				)
+				(hide yes)
+			)
+		)
+		(pin "1"
+		)
+		(pin "2"
+		)
+		(instances
+			(project "neopico-hd"
+				(path "/e43af130-6d9a-4b98-bcf6-f3f51cb37ae8"
+					(reference "R2")
+					(unit 1)
+				)
+			)
+		)
+	)
+	(symbol
 		(lib_id "power:GND")
 		(at 269.24 97.79 0)
@@
 		(on_board yes)
 		(dnp no)
-		(fields_autoplaced yes)
 		(property "Reference" "#PWR034"
 			(at 264.16 104.14 0)
@@
 		)
 		(property "Value" "GND"
-			(at 264.16 102.87 0)
+			(at 261.62 102.87 90)
 			(effects
 				(font
@@
 		(on_board yes)
 		(dnp no)
-		(fields_autoplaced yes)
 		(property "Reference" "#PWR033"
 			(at 261.62 104.14 0)
@@
 		)
 		(property "Value" "GND"
-			(at 261.62 102.87 0)
+			(at 264.16 102.87 90)
 			(effects
 				(font
